Commit message: Full-robot Gazebo sim: shared upper body, simulated camera, measured base
- humanoi_full.urdf.xacro / srdf use ar_dual's humanoi_upper.xacro and
  arm_control.xacro (same arms, hands and controllers as the real robot)
- simulated Astra Pro bridged to the real driver's topic names
  (/camera/color/image_raw, camera_info, depth, points)
- mecanum base dimensions measured
- moveit_full / sim_with_arm launch updated; run_humanoi_gz.bat opens
  Gazebo, MoveIt + RViz and the program player in WSL

Co-Authored-By: Claude Opus 5.5 <noreply@anthropic.com>

File: ros2_ws/src/humanoi_description/srdf/humanoi_full.srdf.xacro (robot description, xacro)
@@ -1,34 +1,16 @@
 <?xml version="1.0" encoding="UTF-8"?>
-<!-- SRDF ของหุ่นรวม (ฐาน mecanum + แขน AR4)
-     ส่วนของแขนทั้งหมด (group ar_manipulator, group_state home/upright, disable_collisions
-     ระหว่างลิงก์แขนด้วยกัน) เรียกจาก macro ของผู้ขายตรงๆ ไม่คัดลอกมาซ้ำ ไม่แก้ไฟล์ผู้ขาย
-     ไฟล์นี้เพิ่มเฉพาะสิ่งที่ "เกิดจากการเอาแขนมาวางบนฐาน" เท่านั้น
+<!-- SRDF ของหุ่นเต็มตัว (ฐาน mecanum + ลำตัวบนสองแขน — urdf/humanoi_full.urdf.xacro)
+     กลุ่ม left_arm / right_arm / both_arms, ท่า rest และคู่ลิงก์ที่ไม่ต้องเช็กชนของแขน/เสา/มือ
+     ดึงจาก SRDF ของระบบแขนจริง (ar_dual/srdf/humanoi_arms.srdf) ตรงๆ ไม่คัดลอกซ้ำ
+     ไฟล์นี้เพิ่มเฉพาะคู่ที่เกิดจากการวางลำตัวบนแผ่นฐาน
        xacro humanoi_full.srdf.xacro -->
 <robot xmlns:xacro="http://wiki.ros.org/xacro" name="humanoi">
-  <xacro:include filename="$(find ar_moveit_config)/srdf/ar_macro.srdf.xacro"/>
-  <xacro:ar_srdf/>
-  <!-- ===== คู่ลิงก์ที่ไม่ต้องเช็คการชน =====
-       ปิดเฉพาะคู่ที่ "ติดกันอยู่แล้วโดยโครงสร้าง" เท่านั้น
-       ตั้งใจ *ไม่* ปิด link_2..link_6 กับ chassis_link/laser_link — อยากให้ MoveIt กันแขน
-       ฟาดลงฝาบนฐานหรือฟาดไลดาร์จริงๆ ซึ่งเป็นประโยชน์หลักอย่างหนึ่งของการรวมโมเดล -->
-  <disable_collisions link1="chassis_link" link2="base_link"  reason="Adjacent"/>
-  <disable_collisions link1="chassis_link" link2="link_1"     reason="Never"/>
-  <disable_collisions link1="chassis_link" link2="laser_link" reason="Adjacent"/>
-  <disable_collisions link1="chassis_link" link2="front_left_wheel"  reason="Adjacent"/>
-  <disable_collisions link1="chassis_link" link2="front_right_wheel" reason="Adjacent"/>
-  <disable_collisions link1="chassis_link" link2="rear_left_wheel"   reason="Adjacent"/>
-  <disable_collisions link1="chassis_link" link2="rear_right_wheel"  reason="Adjacent"/>
-  <!-- ===== ท่าที่ตั้งโปรแกรมไว้ล่วงหน้า =====
-       "stow" = ท่าพับเก็บ ต้องเข้าท่านี้ก่อนฐานจะเคลื่อนที่ทุกครั้ง (กันหุ่นคว่ำ / ฟาดของ)
-       humanoi_mission จะบังคับเงื่อนไขนี้เป็น interlock
-       ⚠️ ค่าด้านล่างยังเป็นค่าตั้งต้น ต้องเปิด RViz ดูด้วยตาว่าแขนพับเก็บจริงก่อนใช้งาน
-          เครื่องหมายของ joint_2/joint_3 ยังไม่ได้ยืนยันด้วยภาพ -->
-  <group_state name="stow" group="ar_manipulator">
-    <joint name="joint_1" value="0"/>
-    <joint name="joint_2" value="1.40"/>
-    <joint name="joint_3" value="-1.50"/>
-    <joint name="joint_4" value="0"/>
-    <joint name="joint_5" value="0"/>
-    <joint name="joint_6" value="0"/>
-  </group_state>
+  <xacro:include filename="$(find ar_dual)/srdf/humanoi_arms.srdf"/>
+  <!-- เสายึดกับแผ่นฐาน · ฐานแขนอยู่สูง 1.45 m แตะแผ่นฐานไม่ได้
+       ยังเช็กแขน/มือกับแผ่นฐานตามปกติ (ล้อกับไลดาร์ไม่มีรูปทรงชน) -->
+  <disable_collisions link1="chassis_link" link2="torso" reason="Adjacent"/>
+  <disable_collisions link1="chassis_link" link2="left_base_link" reason="Never"/>
+  <disable_collisions link1="chassis_link" link2="right_base_link" reason="Never"/>
+  <disable_collisions link1="chassis_link" link2="left_link_1" reason="Never"/>
+  <disable_collisions link1="chassis_link" link2="right_link_1" reason="Never"/>
 </robot>

File: ros2_ws/src/humanoi_description/urdf/humanoi_full.urdf.xacro (robot description, xacro)
@@ -1,103 +1,96 @@
 <?xml version="1.0"?>
-<!-- หุ่น Humanoi ตัวเต็ม = ฐาน mecanum + แขน AR4 หนึ่งข้างบนฝาบน (ไมล์สโตน M16)
-     ประกอบจากของที่มีอยู่แล้วทั้งหมด ไม่แก้ไฟล์ผู้ขายแม้แต่ไฟล์เดียว:
-       - mecanum_base.urdf.xacro    (ของเรา — ฐาน ล้อ ไลดาร์ ปลั๊กอิน gz ของฐาน)
-       - ar_description/ar_macro.xacro  (ของผู้ขาย — ลิงก์/ข้อต่อ/เมช AR4 อ่านอย่างเดียว)
-     เรื่องชื่อลิงก์: ar_macro.xacro ฮาร์ดโค้ดลิงก์รากเป็น "base_link" + joint "base_joint"
-     และไม่มีพารามิเตอร์ prefix ให้ ฐานจึงถูกเปลี่ยนไปใช้ "chassis_link"/"chassis_joint" แทน
-     (เหตุผลเต็มอยู่ในคอมเมนต์ของ mecanum_base.urdf.xacro) แขนคงชื่อเดิมทุกอย่าง
-     SRDF/kinematics/joint_limits ของผู้ขายจึงใช้ต่อได้ตรงๆ ไม่ต้องแก้
-       xacro humanoi_full.urdf.xacro arm_controllers:=/path/to/arm_controllers.yaml
-     ⚠️ ข้อจำกัดที่รู้อยู่: ฐานยังขับด้วยปลั๊กอิน VelocityControl แบบ kinematic (ล้อไม่มี
-        collision ไม่หมุนจริง) ฐานจึงไม่มีปฏิกิริยาต่อน้ำหนักแขนเลย — ยื่นแขนสุดแขนก็ไม่เอียง
-        ไม่คว่ำ ใช้ดู "ท่าหยิบของ" และระยะเอื้อมได้ แต่ยังตอบเรื่องเสถียรภาพ/การคว่ำไม่ได้
-        ต้องรอเฟสล้อจริง (ros2_control ต่อล้อ + ลูกกลิ้ง mecanum) -->
+<!-- หุ่น Humanoi เต็มตัวสำหรับ Gazebo = ฐาน mecanum + เสา หัว กล้อง + แขน AR4 สองข้าง + มือ AmazingHand
+  ประกอบจากไฟล์ที่ใช้กับของจริงทั้งหมด แก้ขนาดที่ต้นทางที่เดียว:
+    - mecanum_base.urdf.xacro         (ของเรา — แผ่นฐาน ล้อ ไลดาร์ ปลั๊กอิน gz ของฐาน)
+    - ar_dual/urdf/humanoi_upper.xacro (ของเรา ใน repo ar4 — เสา หัว กล้อง สองแขน มือ: ไฟล์เดียวกับระบบแขนจริง)
+    - ar_dual/urdf/arm_control.xacro   (ros2_control ต่อแขน — ใช้แบบ gz ที่นี่)
+    - config/camera_to_left_arm.yaml   (ตำแหน่งกล้องจาก hand-eye calibration — ไฟล์เดียวกับที่ yolo.launch.py ใช้)
+    xacro humanoi_full.urdf.xacro
+  แขนสั่งด้วย left_arm_controller / right_arm_controller ชื่อเดียวกับแขนจริง (ar_dual/config/controllers.yaml)
+  MoveIt + ตัวเล่นโปรแกรม (ar_program) จึงใช้กับซิมได้เลยโดยไม่ต้องแก้
+  ⚠️ ฐานยังขับด้วยปลั๊กอิน VelocityControl แบบ kinematic (ล้อไม่หมุนจริง) — ฐานไม่เอียง/ไม่คว่ำ
+     ตามน้ำหนักแขน ใช้ดูท่า ระยะเอื้อม การชน และภาพกล้องได้ แต่ยังตอบเรื่องเสถียรภาพไม่ได้
+-->
 <robot xmlns:xacro="http://wiki.ros.org/xacro" name="humanoi">
-  <xacro:arg name="arm_controllers" default=""/>
-  <!-- ตำแหน่งติดตั้งแขนบนฝาบนของฐาน (แก้ได้เมื่อวัดฐานจริง) -->
-  <xacro:property name="arm_mount_x" value="-0.08"/>
-  <xacro:property name="arm_mount_y" value="0.0"/>
-  <xacro:property name="arm_mount_z" value="0.06"/>   <!-- = base_z/2 คือผิวฝาบน -->
+  <xacro:arg name="controllers" default="$(find ar_dual)/config/controllers.yaml"/>
+  <xacro:arg name="camera_yaml" default="$(find humanoi_description)/config/camera_to_left_arm.yaml"/>
   <xacro:include filename="$(find humanoi_description)/urdf/mecanum_base.urdf.xacro"/>
-  <xacro:include filename="$(find ar_description)/urdf/ar_macro.xacro"/>
-  <!-- แขนเกาะฝาบนของฐาน — ar_robot รับ parent + *origin มาอยู่แล้ว ไม่ต้องดัดแปลงอะไร
-       วางค่อนไปด้านหลังเล็กน้อยเพื่อลดการบังไลดาร์ที่อยู่หน้าฐาน (x = +0.16)
-       หมายเหตุ: ยังบังอยู่บางส่วนอยู่ดี ตอนทำ Nav2 จริงต้องยกไลดาร์ให้สูงกว่าฐานแขน
-       หรือใส่ตัวกรองมุมใน laser_filters ไม่งั้น costmap จะเห็นแขนตัวเองเป็นสิ่งกีดขวาง -->
-  <xacro:ar_robot parent="chassis_link">
-    <origin xyz="${arm_mount_x} ${arm_mount_y} ${arm_mount_z}" rpy="0 0 0"/>
-  </xacro:ar_robot>
-  <!-- ===================== ros2_control ของแขน =====================
-       สำเนาจาก ar_gz_bringup/urdf/ar_gz.urdf.xacro ที่ยืนยันแล้วว่าใช้งานได้จริง
-       (เขียนเองแทนการเรียก xacro:ar_ros2_control ของผู้ขาย เพราะไฟล์นั้น limit เขียนเป็น
-        "{-170*pi/180}" ขาด "$" นำหน้า gz_ros2_control จึง parse ไม่ผ่าน และไม่ได้ตั้ง
-        position_proportional_gain ทำให้ใช้ default 0.1 ซึ่งอ่อนเกินจะต้านแรงโน้มถ่วง
-        แขนค่อยๆห้อยลงจนสุด hard-stop)
-       initial_value ของ joint_2/joint_5 ตั้งตามท่าพักจริงของแขนหลัง calibrate -->
-  <ros2_control name="ar" type="system">
-    <hardware>
-      <plugin>gz_ros2_control/GazeboSimSystem</plugin>
-      <param name="serial_port">None</param>
-      <param name="calibrate">False</param>
-      <param name="position_proportional_gain">20.0</param>
-    </hardware>
-    <joint name="joint_1">
-      <command_interface name="position">
-        <param name="min">-2.967060</param>
-        <param name="max">2.967060</param>
-      </command_interface>
-      <state_interface name="position">
-        <param name="initial_value">0.0</param>
-      </state_interface>
-    </joint>
-    <joint name="joint_2">
-      <command_interface name="position">
-        <param name="min">-0.733038</param>
-        <param name="max">1.570796</param>
-      </command_interface>
-      <state_interface name="position">
-        <param name="initial_value">-0.1019</param>
-      </state_interface>
-    </joint>
-    <joint name="joint_3">
-      <command_interface name="position">
-        <param name="min">-1.553343</param>
-        <param name="max">0.907571</param>
-      </command_interface>
-      <state_interface name="position">
-        <param name="initial_value">0.0</param>
-      </state_interface>
-    </joint>
-    <joint name="joint_4">
-      <command_interface name="position">
-        <param name="min">-2.879793</param>
-        <param name="max">2.879793</param>
-      </command_interface>
-      <state_interface name="position">
-        <param name="initial_value">0.0</param>
-      </state_interface>
-    </joint>
-    <joint name="joint_5">
-      <command_interface name="position">
-        <param name="min">-1.832596</param>
-        <param name="max">1.832596</param>
-      </command_interface>
-      <state_interface name="position">
-        <param name="initial_value">-0.9103</param>
-      </state_interface>
-    </joint>
-    <joint name="joint_6">
-      <command_interface name="position">
-        <param name="min">-2.705260</param>
-        <param name="max">2.705260</param>
-      </command_interface>
-      <state_interface name="position">
-        <param name="initial_value">0.0</param>
-      </state_interface>
-    </joint>
-  </ros2_control>
+  <xacro:include filename="$(find ar_dual)/urdf/humanoi_upper.xacro"/>
+  <xacro:include filename="$(find ar_dual)/urdf/arm_control.xacro"/>
+  <!-- ลำตัวบน: เสาอยู่กึ่งกลางฐานทั้งหน้า-หลัง (หน้าเสาห่างขอบหน้าฐาน 20.5 cm = G, ฐานยาว 51 cm)
+       และซ้าย-ขวา · หัวไหล่สูงจากพื้น up_shoulder_z -->
+  <joint name="torso_joint" type="fixed">
+    <parent link="chassis_link"/>
+    <child link="torso"/>
+    <origin xyz="${-up_pole_dx} 0 ${up_shoulder_z - wheel_radius - clearance}" rpy="0 0 0"/>
+  </joint>
+  <xacro:humanoi_upper left_hand="true" right_hand="true"/>
+  <xacro:arm_control prefix="left_" hw="gz"/>
+  <xacro:arm_control prefix="right_" hw="gz"/>
+  <!-- ===================== กล้อง Astra Pro จำลอง =====================
+       camera_link อยู่ตรงตำแหน่งที่ hand-eye calibration วัดได้ (เทียบฐานแขนซ้าย)
+       ภาพสี 640x480 ค่าเลนส์ที่ calibrate จริง (config/astra_color.yaml): fx 631.98 fy 633.19 cx 321.59 cy 229.81
+       horizontal_fov = 2·atan(320/631.98) — ไม่รวมความบิดเบี้ยวเลนส์ (k1, k2)
+       ความลึก 0.6–8 m เหมือนตัวจริง (ใกล้กว่า 0.6 m วัดไม่ได้)
+       สมมติว่าเฟรมภาพสีของไดรเวอร์จริงทับกับ camera_link (ไดรเวอร์ไม่มีค่าโรงงานของกล้องตัวนี้) -->
+  <xacro:property name="cam_file" value="$(arg camera_yaml)"/>
+  <xacro:property name="cam" value="${xacro.load_yaml(cam_file)}"/>
+  <xacro:property name="cam_roll"
+    value="${atan2(2 * (cam['qw'] * cam['qx'] + cam['qy'] * cam['qz']), 1 - 2 * (cam['qx'] ** 2 + cam['qy'] ** 2))}"/>
+  <xacro:property name="cam_pitch"
+    value="${asin(max(-1.0, min(1.0, 2 * (cam['qw'] * cam['qy'] - cam['qz'] * cam['qx']))))}"/>
+  <xacro:property name="cam_yaw"
+    value="${atan2(2 * (cam['qw'] * cam['qz'] + cam['qx'] * cam['qy']), 1 - 2 * (cam['qy'] ** 2 + cam['qz'] ** 2))}"/>
+  <joint name="camera_joint" type="fixed">
+    <parent link="${cam['parent_frame']}"/>
+    <child link="camera_link"/>
+    <origin xyz="${cam['x']} ${cam['y']} ${cam['z']}" rpy="${cam_roll} ${cam_pitch} ${cam_yaw}"/>
+  </joint>
+  <link name="camera_link"/>
+  <joint name="camera_color_optical_joint" type="fixed">
+    <parent link="camera_link"/>
+    <child link="camera_color_optical_frame"/>
+    <origin xyz="0 0 0" rpy="${-pi / 2} 0 ${-pi / 2}"/>
+  </joint>
+  <link name="camera_color_optical_frame"/>
+  <gazebo reference="camera_link">
+    <!-- gz มองตามแกน +X ของ camera_link · ข้อความใน ROS ใช้เฟรม optical แบบเดียวกับไดรเวอร์จริง -->
+    <sensor name="astra" type="rgbd_camera">
+      <update_rate>15</update_rate>
+      <always_on>1</always_on>
+      <topic>camera</topic>
+      <gz_frame_id>camera_color_optical_frame</gz_frame_id>
+      <camera>
+        <horizontal_fov>0.93742</horizontal_fov>
+        <image>
+          <width>640</width>
+          <height>480</height>
+          <format>R8G8B8</format>
+        </image>
+        <lens>
+          <intrinsics>
+            <fx>631.98</fx>
+            <fy>633.19</fy>
+            <cx>321.59</cx>
+            <cy>229.81</cy>
+            <s>0</s>
+          </intrinsics>
+        </lens>
+        <clip>
+          <near>0.05</near>
+          <far>10.0</far>
+        </clip>
+        <depth_camera>
+          <clip>
+            <near>0.6</near>
+            <far>8.0</far>
+          </clip>
+        </depth_camera>
+      </camera>
+    </sensor>
+  </gazebo>
   <gazebo>
     <plugin filename="gz_ros2_control-system" name="gz_ros2_control::GazeboSimROS2ControlPlugin">
-      <parameters>$(arg arm_controllers)</parameters>
+      <parameters>$(arg controllers)</parameters>
     </plugin>
   </gazebo>

File: ros2_ws/src/humanoi_description/urdf/mecanum_base.urdf.xacro (robot description, xacro)
@@ -1,21 +1,28 @@
 <?xml version="1.0"?>
 <!-- ฐานหุ่น Humanoi : 4 ล้อ mecanum ขับเคลื่อนแบบ holonomic
-     ค่าทั้งหมดปรับได้ที่บล็อก property ด้านล่าง (ยังเป็นค่าสมมติจนกว่าจะวัดฐานจริง)
+     ค่าทั้งหมดปรับได้ที่บล็อก property ด้านล่าง (วัดจริงแล้วบางส่วน — ดูหมายเหตุแต่ละค่า)
      หมายเหตุ sim: ใช้ปลั๊กอิน VelocityControl (ขยับตัวถังตาม /cmd_vel ตรงๆ แบบ kinematic)
      ไม่ได้ขับผ่านแรงเสียดทานล้อ เพราะล้อทรงกระบอกไม่มีลูกกลิ้ง mecanum จริง จึงสไลด์ข้างไม่ได้
      ล้อในโมเดลจึงเป็นแค่ visual (ยังไม่หมุนตาม) — odom มาจากตำแหน่งจริงของหุ่น -->
 <robot name="humanoi_base" xmlns:xacro="http://www.ros.org/wiki/xacro">
-  <!-- ===================== ค่าที่ปรับได้ ===================== -->
-  <xacro:property name="base_x"    value="0.45"/>   <!-- ยาว (หน้า-หลัง) เมตร -->
-  <xacro:property name="base_y"    value="0.35"/>   <!-- กว้าง (ซ้าย-ขวา) เมตร -->
-  <xacro:property name="base_z"    value="0.12"/>   <!-- สูงของกล่องฐาน เมตร -->
-  <xacro:property name="base_mass" value="14.0"/>   <!-- กก. (ประมาณ ฐาน+แบต) -->
-  <xacro:property name="wheel_radius" value="0.075"/>  <!-- ล้อ Ø150 mm -->
-  <xacro:property name="wheel_width"  value="0.05"/>
+  <!-- ===================== ค่าที่ปรับได้ =====================
+       วัดจากหุ่นจริง 19 ต.ค. 2026: ยาวฐาน (A), ความหนาแผ่นฐาน (B), พื้น->ใต้แผ่น (C), ล้อ Ø (D), ไลดาร์สูง (F)
+       ค่าที่เขียนว่า "ยังไม่ได้วัด" เป็นค่าประมาณ -->
+  <xacro:property name="base_x"    value="0.51"/>   <!-- A: ยาว (หน้า-หลัง) -->
+  <xacro:property name="base_y"    value="0.40"/>   <!-- กว้าง (ซ้าย-ขวา) — ยังไม่ได้วัด -->
+  <xacro:property name="base_z"    value="0.01"/>   <!-- B: ฐานเป็นแผ่นหนา 1 cm -->
+  <xacro:property name="plate_bottom" value="0.195"/> <!-- C: พื้น -> ใต้แผ่นฐาน -->
+  <xacro:property name="base_mass" value="14.0"/>   <!-- กก. (ประมาณ ฐาน+แบต) — ยังไม่ได้ชั่ง -->
+  <xacro:property name="wheel_radius" value="0.075"/>  <!-- D: ล้อ Ø150 mm -->
+  <xacro:property name="wheel_width"  value="0.05"/>   <!-- ยังไม่ได้วัด -->
   <xacro:property name="wheel_mass"   value="0.6"/>
-  <!-- ระยะติดตั้งล้อ วัดจากจุดศูนย์กลางฐาน (ครึ่งระยะ) -->
-  <xacro:property name="track_half"     value="0.20"/>  <!-- ครึ่งระยะ ซ้าย-ขวา ระหว่างล้อ -->
-  <xacro:property name="wheelbase_half" value="0.16"/>  <!-- ครึ่งระยะ หน้า-หลัง ระหว่างล้อ -->
-  <xacro:property name="clearance"      value="0.04"/>  <!-- ระยะกล่องฐานลอยเหนือแกนล้อ -->
+  <!-- ระยะติดตั้งล้อ วัดจากจุดศูนย์กลางฐาน (ครึ่งระยะ) — ยังไม่ได้วัดทั้งคู่ -->
+  <xacro:property name="track_half"     value="0.20"/>  <!-- ครึ่งระยะ ซ้าย-ขวา ระหว่างกลางล้อ -->
+  <xacro:property name="wheelbase_half" value="0.17"/>  <!-- ครึ่งระยะ หน้า-หลัง ระหว่างแกนล้อ -->
+  <!-- แกนล้อ -> กึ่งกลางแผ่นฐาน (คำนวณจาก C, B, D) -->
+  <xacro:property name="clearance" value="${plate_bottom + base_z / 2 - wheel_radius}"/>
+  <!-- ไลดาร์ LDROBOT STL-19P: สูงจากพื้นถึงกลางตัว 22.25 cm (F) วางบนแผ่นฐาน -->
+  <xacro:property name="lidar_z" value="0.2225"/>
+  <xacro:property name="lidar_x" value="0.16"/>     <!-- หน้าเสา ค่อนไปขอบหน้า — ยังไม่ได้วัด -->
   <!-- ======================================================= -->
   <material name="hull">   <color rgba="0.90 0.50 0.10 1"/></material>
@@ -41,4 +48,16 @@
       <material name="hull"/>
     </visual>
+    <!-- ขายึดมอเตอร์ล้อใต้แผ่นฐาน (ดูอย่างเดียว ขนาดประมาณ) — แผ่นอยู่สูงกว่ายอดล้อ 4.5 cm -->
+    <xacro:macro name="wheel_bracket" params="x y">
+      <visual>
+        <origin xyz="${x} ${y} ${-(clearance + base_z / 2) / 2}" rpy="0 0 0"/>
+        <geometry><box size="0.06 0.03 ${clearance - base_z / 2}"/></geometry>
+        <material name="rubber"/>
+      </visual>
+    </xacro:macro>
+    <xacro:wheel_bracket x="${ wheelbase_half}" y="${ track_half - wheel_width / 2 - 0.02}"/>
+    <xacro:wheel_bracket x="${ wheelbase_half}" y="${-track_half + wheel_width / 2 + 0.02}"/>
+    <xacro:wheel_bracket x="${-wheelbase_half}" y="${ track_half - wheel_width / 2 - 0.02}"/>
+    <xacro:wheel_bracket x="${-wheelbase_half}" y="${-track_half + wheel_width / 2 + 0.02}"/>
     <collision>
       <geometry><box size="${base_x} ${base_y} ${base_z}"/></geometry>
@@ -52,6 +71,8 @@
     </inertial>
   </link>
-  <!-- ล้อ 1 ตัว : visual + inertial เท่านั้น (ไม่มี collision — ดูหมายเหตุด้านบน)
-       ศูนย์กลางล้ออยู่สูง wheel_radius จากพื้น -> ล้อแตะพื้นพอดี -->
+  <!-- ล้อ 1 ตัว : ศูนย์กลางล้ออยู่สูง wheel_radius จากพื้น -> ล้อแตะพื้นพอดี
+       collision เป็นทรงกลมไร้แรงเสียดทาน (mu = 0) แค่รองรับน้ำหนักให้หุ่นยืนบนพื้น
+       (VelocityControl ไม่ล็อกแกน Z — ถ้าไม่มีอะไรรับ หุ่นจะร่วงจนแผ่นฐานแตะพื้น)
+       ไร้แรงเสียดทานเพื่อไม่ให้ล้อทรงกลม/กระบอกไปฝืนการสไลด์ข้างของ VelocityControl -->
   <xacro:macro name="wheel" params="name x y">
     <link name="${name}_wheel">
@@ -61,4 +82,7 @@
         <material name="rubber"/>
       </visual>
+      <collision>
+        <geometry><sphere radius="${wheel_radius}"/></geometry>
+      </collision>
       <inertial>
         <mass value="${wheel_mass}"/>
@@ -76,4 +100,8 @@
       <dynamics damping="0.05" friction="0.0"/>
     </joint>
+    <gazebo reference="${name}_wheel">
+      <mu1>0.0</mu1>
+      <mu2>0.0</mu2>
+    </gazebo>
   </xacro:macro>
   <xacro:wheel name="front_left"  x="${ wheelbase_half}" y="${ track_half}"/>
@@ -100,6 +128,5 @@
     <parent link="chassis_link"/>
     <child  link="laser_link"/>
-    <!-- กลางฐาน ค่อนไปหน้า สูงพ้นฝาบน -->
-    <origin xyz="${wheelbase_half} 0 ${base_z/2 + 0.04}" rpy="0 0 0"/>
+    <origin xyz="${lidar_x} 0 ${lidar_z - wheel_radius - clearance}" rpy="0 0 0"/>
   </joint>
   <gazebo reference="laser_link">
