Commit message: Measured base size: 53 x 42.5 cm, wheels 14.5 cm x 4 cm
- track = 42.5 - 4 = 38.5 cm, wheelbase = 53 - 14.5 = 38.5 cm (wheels are the
  outermost points), wheel radius 0.0725
- mecanum_base.urdf.xacro, relay_bridge defaults + config/base.yaml (odometry),
  lidar guard footprint 0.265 / 0.2125 m, nav2 robot_radius 0.35
- lidar position is still the 0.16 m guess

Co-Authored-By: Claude Opus 5.5 <noreply@anthropic.com>

File: ros2_ws/src/humanoi_description/urdf/mecanum_base.urdf.xacro (robot description, xacro)
@@ -14,10 +14,11 @@
   <xacro:property name="plate_bottom" value="0.195"/> <!-- C: พื้น -> ใต้แผ่นฐาน -->
   <xacro:property name="base_mass" value="14.0"/>   <!-- กก. (ประมาณ ฐาน+แบต) — ยังไม่ได้ชั่ง -->
-  <xacro:property name="wheel_radius" value="0.075"/>  <!-- D: ล้อ Ø150 mm -->
-  <xacro:property name="wheel_width"  value="0.05"/>   <!-- ยังไม่ได้วัด -->
+  <xacro:property name="wheel_radius" value="0.0725"/> <!-- D: ล้อ Ø145 mm (วัด 28 ต.ค.) -->
+  <xacro:property name="wheel_width"  value="0.04"/>   <!-- หนา 4 cm (วัดแล้ว) -->
   <xacro:property name="wheel_mass"   value="0.6"/>
-  <!-- ระยะติดตั้งล้อ วัดจากจุดศูนย์กลางฐาน (ครึ่งระยะ) — ยังไม่ได้วัดทั้งคู่ -->
-  <xacro:property name="track_half"     value="0.20"/>  <!-- ครึ่งระยะ ซ้าย-ขวา ระหว่างกลางล้อ -->
-  <xacro:property name="wheelbase_half" value="0.17"/>  <!-- ครึ่งระยะ หน้า-หลัง ระหว่างแกนล้อ -->
+  <!-- ระยะติดตั้งล้อ วัดจากจุดศูนย์กลางฐาน (ครึ่งระยะ) — คำนวณจากที่วัด 28 ต.ค.:
+       กว้างรวมนอกล้อ 42.5 cm − ล้อหนา 4 = 38.5 · ยาวรวม 53 cm (ล้อยื่นสุด) − ล้อ Ø14.5 = 38.5 -->
+  <xacro:property name="track_half"     value="0.1925"/>  <!-- ครึ่งระยะ ซ้าย-ขวา ระหว่างกลางล้อ -->
+  <xacro:property name="wheelbase_half" value="0.1925"/>  <!-- ครึ่งระยะ หน้า-หลัง ระหว่างแกนล้อ -->
   <!-- แกนล้อ -> กึ่งกลางแผ่นฐาน (คำนวณจาก C, B, D) -->
   <xacro:property name="clearance" value="${plate_bottom + base_z / 2 - wheel_radius}"/>

Commit message: Lidar height 23.5 cm (measured), guard test teardown fix
- lidar.launch standalone TF and mecanum_base.urdf.xacro lidar_z = 0.235
- BASE_SAFETY.md: what a 23.5 cm scan plane can and cannot see
- test_guard_e2e.py: join the spin thread before rclpy shutdown (aborted
  at exit on the Pi even though all checks passed)

Co-Authored-By: Claude Opus 5.5 <noreply@anthropic.com>

File: ros2_ws/src/humanoi_description/urdf/mecanum_base.urdf.xacro (robot description, xacro)
@@ -23,6 +23,6 @@
   <!-- แกนล้อ -> กึ่งกลางแผ่นฐาน (คำนวณจาก C, B, D) -->
   <xacro:property name="clearance" value="${plate_bottom + base_z / 2 - wheel_radius}"/>
-  <!-- ไลดาร์ LDROBOT STL-19P: สูงจากพื้นถึงกลางตัว 22.25 cm (F) วางบนแผ่นฐาน -->
-  <xacro:property name="lidar_z" value="0.2225"/>
+  <!-- ไลดาร์ LDROBOT STL-19P: สูงจากพื้น 23.5 cm (วัดหุ่นจริง 29 ต.ค.) วางบนแผ่นฐาน -->
+  <xacro:property name="lidar_z" value="0.235"/>
   <xacro:property name="lidar_x" value="0.16"/>     <!-- หน้าเสา ค่อนไปขอบหน้า — ยังไม่ได้วัด -->
   <!-- ======================================================= -->

Commit message: Lidar sits 17.5 cm ahead of the base centre (measured, was a 16 cm guess)
Measured on the robot: lidar centre to base plate front edge 2.5 cm, rear
37.5 cm (left 15.5, right 15 — 2.5 mm off centre, ignored). One constant
LIDAR_X in base_motion now feeds the no-TF fallbacks of base_motion, the
guard and scan_mask; lidar.launch and the xacro carry the same value.

Co-Authored-By: Claude Opus 5.5 <noreply@anthropic.com>

File: ros2_ws/src/humanoi_description/urdf/mecanum_base.urdf.xacro (robot description, xacro)
@@ -25,5 +25,5 @@
   <!-- ไลดาร์ LDROBOT STL-19P: สูงจากพื้น 23.5 cm (วัดหุ่นจริง 29 ต.ค.) วางบนแผ่นฐาน -->
   <xacro:property name="lidar_z" value="0.235"/>
-  <xacro:property name="lidar_x" value="0.16"/>     <!-- หน้าเสา ค่อนไปขอบหน้า — ยังไม่ได้วัด -->
+  <xacro:property name="lidar_x" value="0.175"/>    <!-- กลาง lidar ถึงขอบแผ่นฐานหน้า 2.5 หลัง 37.5 cm (วัด 29 ต.ค.) -->
   <!-- ======================================================= -->
   <material name="hull">   <color rgba="0.90 0.50 0.10 1"/></material>

Commit message: arm lidar-check: measure lidar yaw and catch a mirrored scan
The lidar pose now lives in one file, humanoi_base/config/lidar_mount.yaml
(x, y, z, yaw_deg). lidar.launch takes its static TF and scan_mask
defaults from it, and the guard and base_motion use it when there is no TF.

lidar_check: a narrow upright object on the base centreline about 1 m
ahead must show at 0 deg in the raw scan; any offset is the mounting yaw
and is saved to lidar_mount.yaml. Moving the object to the robot's left
must make new points appear at a positive angle; otherwise the scan is
mirrored, which would make the guard block the wrong side, and nothing is
saved. A 5 s countdown lets the operator step out of the scan first.
wheel-check and lidar-check chown the YAML they write from the container.

Co-Authored-By: Claude Opus 5.5 <noreply@anthropic.com>

File: ros2_ws/src/humanoi_description/urdf/mecanum_base.urdf.xacro (robot description, xacro)
@@ -25,5 +25,5 @@
   <!-- ไลดาร์ LDROBOT STL-19P: สูงจากพื้น 23.5 cm (วัดหุ่นจริง 29 ต.ค.) วางบนแผ่นฐาน -->
   <xacro:property name="lidar_z" value="0.235"/>
-  <xacro:property name="lidar_x" value="0.175"/>    <!-- กลาง lidar ถึงขอบแผ่นฐานหน้า 2.5 หลัง 37.5 cm (วัด 29 ต.ค.) -->
+  <xacro:property name="lidar_x" value="0.175"/>    <!-- เท่า humanoi_base/config/lidar_mount.yaml (หุ่นจริง) -->
   <!-- ======================================================= -->
   <material name="hull">   <color rgba="0.90 0.50 0.10 1"/></material>
